File: 0010_PIR_Module_LHI778.kicad_sch (KiCad schematic)
At the start: 30 parts, among them J1 Conn_01x03_Female, Q1 BC546, T1 1m, U1 LHI778, U2 BISS0001

Commit message: Add files via upload
Parts:
- added U3: ~, Moduler_:pin_header, symbol moduler_pin:air
- C1, C2, C3, C4, C6: footprint (none) -> Capacitor_SMD:C_0603_1608Metric
- C10, C5, C7, C9: footprint (none) -> Capacitor_Tantalum_SMD:CP_EIA-1608-08_AVX-J
- C8: footprint (none) -> Capacitor_SMD:C_0603_1608Metric_Pad1.08x0.95mm_HandSolder
- D1: footprint (none) -> LED_SMD:LED_0603_1608Metric
- J1: footprint (none) -> Jumper:SolderJumper-3_P1.3mm_Open_Pad1.0x1.5mm_NumberLabels
- Q1: footprint Package_TO_SOT_THT:TO-92_Inline -> Package_TO_SOT_SMD:SOT-23
- R1, R10, R11, R12, R13, R14, R2, R3, R4, R6, R7, R8, R9: footprint (none) -> Resistor_SMD:R_0603_1608Metric
- T1: footprint (none) -> memin:3362P_1
- U1: footprint SNR3-D8.1XH4.2MM -> pir:SNR3-D8.1XH4.2MM
- U2: footprint SOIC127P600X180-16N -> pir:SOIC127P600X180-16N
Connections:
- net +3V3: now also U3.8
- net EN: now also U3.14
- net GND: now also U3.9
- net OUT: now also U3.13
- net SIG: now also U3.12
- no-connect marks 0 -> 13
Other:
- note added: "AIR PIN"
- note added: "SENSOR"
- moved on the sheet: C1, C10, C2, C3, C4, C5, C6, C7, C8, C9, D1, J1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
